File: _saved_antdroid-board.sch (KiCad schematic (older format))
At the start: 57 parts, among them P1 CONN_01X01, P2 CONN_01X01, Q1 BSS138, Q2 BSS138, U1 LM2678T-5.0, U2 LM2678T-5.0, U3 LM2675M-5

Commit message: Create lib dir
Parts:
- U1: Suppler http://futurlec.com/ -> (none); Suppler ref LM2678T-5 -> (none); Supplier and ref (none) -> LM2678T-5
- U2: Suppler http://futurlec.com -> (none); Suppler ref LM2678T-5 -> (none); Supplier and ref (none) -> http://futurlec.com
Changed lines of the file:
@@
 F 2 "Power_Integrations:TO-220-7C" H 8850 850 50  0001 C CIN
 F 3 "www.ti.com/lit/ds/symlink/lm2678.pdf" H 8550 1200 50  0001 C CNN
-F 4 "http://futurlec.com/" H 8550 1200 60  0001 C CNN "Suppler"
-F 5 "LM2678T-5" H 8550 1200 60  0001 C CNN "Suppler ref"
+F 4 "LM2678T-5" H 8550 1200 60  0001 C CNN "Supplier and ref"
 	1    8550 1200
 	1    0    0    -1
@@
 F 2 "Power_Integrations:TO-220-7C" H 8850 2200 50  0001 C CIN
 F 3 "www.ti.com/lit/ds/symlink/lm2678.pdf" H 8550 2550 50  0001 C CNN
-F 4 "http://futurlec.com" H 8550 2550 60  0001 C CNN "Suppler"
-F 5 "LM2678T-5" H 8550 2550 60  0001 C CNN "Suppler ref"
+F 4 "http://futurlec.com" H 8550 2550 60  0001 C CNN "Supplier and ref"
 	1    8550 2550
 	1    0    0    -1
