File: antdroid-board.kicad_pcb (KiCad board)
At the start: 2 copper layers, 99.4 x 53.7 mm, 60 parts, among them P1 CONN_01X01, P2 CONN_01X01, Q1 BSS138, Q2 BSS138, U1 LM2678T-5.0, U2 LM2678T-5.0, U3 LM2675M-5

Commit message: LED resistor change to 1K
Parts:
- R1: value 31.2K -> 33K
- R7, R8: value 150Ω -> 1KΩ
Changed lines of the file:
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@@
   )
   (setup
-    (last_trace_width 1)
+    (last_trace_width 0.25)
     (user_trace_width 0.25)
     (user_trace_width 0.6)
@@
       (effects (font (size 1 1) (thickness 0.15)))
     )
-    (fp_text value 31.2K (at 0 1.9) (layer F.Fab)
+    (fp_text value 33K (at 0 1.9) (layer F.Fab)
       (effects (font (size 1 1) (thickness 0.15)))
     )
@@
       (effects (font (size 1 1) (thickness 0.15)))
     )
-    (fp_text value 150Ω (at 0 1.9) (layer F.Fab)
+    (fp_text value 1KΩ (at 0 1.9) (layer F.Fab)
       (effects (font (size 1 1) (thickness 0.15)))
     )
@@
       (effects (font (size 1 1) (thickness 0.15)))
     )
-    (fp_text value 150Ω (at 0 1.9 270) (layer F.Fab)
-      (effects (font (size 1 1) (thickness 0.15)))
-    )
+    (fp_text value 1KΩ (at 0 1.9 270) (layer F.Fab)
+      (effects (font (size 1 1) (thickness 0.15)))
+    )
